File: board/1240pi-rompack-proto/bus_iop.kicad_sch (KiCad schematic)
At the start: 16 parts, among them J30 62684-50210

Commit message: Fully route IO processor lines.
Parts:
- added R31, R32: (no value), symbol Device:R
- added U35: (no value), symbol 74xGxx:74LVC1G32
- added U36: 74LVC1G07, symbol 74xGxx:74LVC1G07
Connections:
- net IO_~{IORQ} is gone; now on net IO_~{IOREQ}: J30.42 (Pin_42)
- net +3V3: now also R31.1, R32.1, U35.5 (VCC), U36.5 (VCC)
- net GND: now also J33.14 (Pin_14), J33.18 (Pin_18), U35.3 (GND), U36.3 (GND)
- net IOB_~{BUSACK}: now also J33.11 (Pin_11), U30.1 (A->B), U31.1 (A->B), U34.1 (A->B), U35.1; no longer J33.9 (Pin_9)
- net IOB_~{CLK}: now also J33.16 (Pin_16); no longer J33.11 (Pin_11)
- net IOB_~{WR}: now also R31.2, U35.2
- net IO_~{BUSACK}: now also R30.2
- net at U32.1 (A->B): now also U35.4
- net IO_~{BUSRQ} renamed IO_~{BUSREQ}
- net IO_~{BUSREQ}: now also U36.4
- removed net ~{CTL_EN}: R30.2, U30.1 (A->B), U31.1 (A->B), U34.1 (A->B)
- new net IOB_~{BUSREQ}: J33.9 (Pin_9), R32.2, U36.2
Other:
- moved on the sheet: R30

Commit message: Add 3.3v regulator.
Parts:
- added C35, C36: (no value), symbol Device:C_Small
Connections:
- net +3V3: now also C35.1, C36.1
- net GND: now also C35.2, C36.2
Changed lines of the file:
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@@
     (pin "2")
+  )
+  (symbol (lib_id "power:+3V3") (at 87.63 175.26 0) (unit 1)
+    (in_bom yes) (on_board yes)
+    (property "Reference" "#PWR0175" (id 0) (at 87.63 179.07 0)
+      (effects (font (size 1.27 1.27)) hide)
+    )
+    (property "Value" "+3V3" (id 1) (at 87.63 171.704 0))
+    (property "Footprint" "" (id 2) (at 87.63 175.26 0)
+      (effects (font (size 1.27 1.27)) hide)
+    )
+    (property "Datasheet" "" (id 3) (at 87.63 175.26 0)
+      (effects (font (size 1.27 1.27)) hide)
+    )
+    (pin "1")
   )
   (symbol (lib_id "power:GND") (at 44.45 58.42 270) (unit 1)
@@
     )
     (property "Datasheet" "~" (id 3) (at 152.4 25.4 0)
+      (effects (font (size 1.27 1.27)) hide)
+    )
+    (pin "1")
+    (pin "2")
+  )
+  (symbol (lib_id "Device:C_Small") (at 184.15 22.86 0) (unit 1)
+    (in_bom yes) (on_board yes)
+    (property "Reference" "C36" (id 0) (at 184.404 21.082 0)
+      (effects (font (size 1.27 1.27)) (justify left))
+    )
+    (property "Value" "" (id 1) (at 184.404 24.892 0)
+      (effects (font (size 1.27 1.27)) (justify left))
+    )
+    (property "Footprint" "" (id 2) (at 184.15 22.86 0)
+      (effects (font (size 1.27 1.27)) hide)
+    )
+    (property "Datasheet" "~" (id 3) (at 184.15 22.86 0)
       (effects (font (size 1.27 1.27)) hide)
     )
@@
     (pin "2")
   )
+  (symbol (lib_id "Device:C_Small") (at 87.63 177.8 0) (unit 1)
+    (in_bom yes) (on_board yes)
+    (property "Reference" "C35" (id 0) (at 87.884 176.022 0)
+      (effects (font (size 1.27 1.27)) (justify left))
+    )
+    (property "Value" "" (id 1) (at 87.884 179.832 0)
+      (effects (font (size 1.27 1.27)) (justify left))
+    )
+    (property "Footprint" "" (id 2) (at 87.63 177.8 0)
+      (effects (font (size 1.27 1.27)) hide)
+    )
+    (property "Datasheet" "~" (id 3) (at 87.63 177.8 0)
+      (effects (font (size 1.27 1.27)) hide)
+    )
+    (pin "1")
+    (pin "2")
+  )
   (symbol (lib_id "power:GND") (at 241.3 25.4 90) (unit 1)
     (in_bom yes) (on_board yes)
@@
     (pin "9")
   )
+  (symbol (lib_id "power:GND") (at 87.63 180.34 0) (unit 1)
+    (in_bom yes) (on_board yes)
+    (property "Reference" "#PWR0174" (id 0) (at 87.63 186.69 0)
+      (effects (font (size 1.27 1.27)) hide)
+    )
+    (property "Value" "GND" (id 1) (at 87.63 184.15 0))
+    (property "Footprint" "" (id 2) (at 87.63 180.34 0)
+      (effects (font (size 1.27 1.27)) hide)
+    )
+    (property "Datasheet" "" (id 3) (at 87.63 180.34 0)
+      (effects (font (size 1.27 1.27)) hide)
+    )
+    (pin "1")
+  )
   (symbol (lib_id "power:GND") (at 62.23 190.5 0) (unit 1)
     (in_bom yes) (on_board yes)
@@
     (pin "2")
   )
+  (symbol (lib_id "power:+3V3") (at 184.15 20.32 0) (unit 1)
+    (in_bom yes) (on_board yes)
+    (property "Reference" "#PWR0176" (id 0) (at 184.15 24.13 0)
+      (effects (font (size 1.27 1.27)) hide)
+    )
+    (property "Value" "+3V3" (id 1) (at 184.15 16.764 0))
+    (property "Footprint" "" (id 2) (at 184.15 20.32 0)
+      (effects (font (size 1.27 1.27)) hide)
+    )
+    (property "Datasheet" "" (id 3) (at 184.15 20.32 0)
+      (effects (font (size 1.27 1.27)) hide)
+    )
+    (pin "1")
+  )
+  (symbol (lib_id "power:GND") (at 184.15 25.4 0) (unit 1)
+    (in_bom yes) (on_board yes)
+    (property "Reference" "#PWR0177" (id 0) (at 184.15 31.75 0)
+      (effects (font (size 1.27 1.27)) hide)
+    )
+    (property "Value" "GND" (id 1) (at 184.15 29.21 0))
+    (property "Footprint" "" (id 2) (at 184.15 25.4 0)
+      (effects (font (size 1.27 1.27)) hide)
+    )
+    (property "Datasheet" "" (id 3) (at 184.15 25.4 0)
+      (effects (font (size 1.27 1.27)) hide)
+    )
+    (pin "1")
+  )
   (symbol (lib_id "power:+3V3") (at 127 46.99 0) (unit 1)

Commit message: Fix names of BUSRQ and IORQ nets.
Parts:
- C30, C31, C32, C33, C34, C35, C36: value (none) -> 2u2; footprint (none) -> Capacitor_SMD:C_0603_1608Metric
- J31, J33: value (none) -> Conn_02x09; footprint (none) -> Connector_PinHeader_2.54mm:PinHeader_2x09_P2.54mm_Vertical
- J32, J34: value (none) -> Conn_01x09; footprint (none) -> Connector_PinHeader_2.54mm:PinHeader_1x09_P2.54mm_Vertical
- R30, R31, R32: value (none) -> 10k; footprint (none) -> Resistor_SMD:R_0603_1608Metric
- U30, U31, U32, U33, U34: value (none) -> 74LVC245A; footprint (none) -> Package_SO:TSSOP-20_4.4x6.5mm_P0.65mm
- U35: value (none) -> 74LVC1G32; footprint (none) -> Package_TO_SOT_SMD:SOT-353_SC-70-5
- U36: footprint (none) -> 0Local:Package_SC-74A
Connections:
- net GND: now also J33.16 (Pin_16); no longer J33.14 (Pin_14)
- net IOB_~{BUSACK}: now also J33.9 (Pin_9); no longer J33.11 (Pin_11)
- net IOB_~{CLK}: now also J33.11 (Pin_11); no longer J33.16 (Pin_16)
- net IOB_~{BUSREQ} renamed IOB_~{BUSRQ}
- net IOB_~{BUSRQ}: now also J33.14 (Pin_14); no longer J33.9 (Pin_9)
- net IOB_~{IOREQ} renamed IOB_~{IORQ}
- net IO_~{BUSREQ} renamed IO_~{BUSRQ}
- net IO_~{IOREQ} renamed IO_~{IORQ}
