File: board/1240pi-rompack-proto/1240pi-rompack-proto.kicad_pcb (KiCad board)
At the start: 2 copper layers, 76.2 x 97.8 mm, 41 parts, among them J20 CardEdge_ROMPACK, J21 Conn_02x09, J22 Conn_01x09, J23 Conn_01x09, J30 62684-50210, J31 Conn_02x09, J32 Conn_01x09, J33 Conn_02x09, J34 Conn_01x09, U10 AMS1117-3.3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

Commit message: Export boards for manufacturing.
Other:
- board text added: "JLCJLCJLCJLC"
Changed lines of the file:
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@@
       (outputformat 1)
       (mirror false)
-      (drillshape 1)
+      (drillshape 0)
       (scaleselection 1)
-      (outputdirectory "")
+      (outputdirectory "${KIPRJMOD}/dist")
     )
   )
@@
     (effects (font (size 1 1) (thickness 0.15)) (justify left))
   )
+  (gr_text "JLCJLCJLCJLC" (at 154.94 72.39) (layer "F.SilkS")
+    (effects (font (size 1 1) (thickness 0.15)))
+  )
   (gr_text "~{EXT}" (at 179.324 154.93) (layer "F.SilkS")
