File: board/proto-hdmi/hdmi_out.kicad_sch (KiCad schematic)
At the start: 30 parts, among them J3 HDMI_A, U2 NXP_NTS0302, U5 MIC2097-1, U6 74LVC1G17

Commit message: Fix 1G17QDRY pinout.
Parts:
- U6: symbol 74xGxx:74LVC1G17 -> 0Local:74LVC1G17QDRY
Connections:
- net +3V3: now also U6.6
- net VCC: no longer names the net of U6.5
Other:
- company: © 2022 Sam Hanes, licensed under CERN-OHL-P v2 -> © 2022 Sam Hanes, licensed under CERN-OHL-S v2
Changed lines of the file:
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@@
   (title_block
     (title "HDMI Expansion for Olimex ICE40HX8K-EVB")
-    (date "2022-04-19")
-    (rev "0.1")
-    (company "© 2022 Sam Hanes, licensed under CERN-OHL-P v2")
+    (date "2022-08-04")
+    (rev "0.2")
+    (company "© 2022 Sam Hanes, licensed under CERN-OHL-S v2")
     (comment 1 "https://github.com/Elemecca/1240pi")
   )
@@
     (effects (font (size 1.27 1.27)) (justify right))
   )
+  (symbol (lib_id "power:+3V3") (at 236.22 168.91 0) (unit 1)
+    (in_bom yes) (on_board yes)
+    (property "Reference" "#PWR0131" (id 0) (at 236.22 172.72 0)
+      (effects (font (size 1.27 1.27)) hide)
+    )
+    (property "Value" "+3V3" (id 1) (at 234.95 165.1 0))
+    (property "Footprint" "" (id 2) (at 236.22 168.91 0)
+      (effects (font (size 1.27 1.27)) hide)
+    )
+    (property "Datasheet" "" (id 3) (at 236.22 168.91 0)
+      (effects (font (size 1.27 1.27)) hide)
+    )
+    (pin "1")
+  )
   (symbol (lib_id "power:GND") (at 233.68 91.44 0) (mirror y) (unit 1)
     (in_bom yes) (on_board yes) (fields_autoplaced)
@@
     (pin "1")
     (pin "2")
+  )
+  (symbol (lib_id "power:GND") (at 236.22 176.53 0) (unit 1)
+    (in_bom yes) (on_board yes) (fields_autoplaced)
+    (property "Reference" "#PWR0130" (id 0) (at 236.22 182.88 0)
+      (effects (font (size 1.27 1.27)) hide)
+    )
+    (property "Value" "GND" (id 1) (at 236.22 181.61 0))
+    (property "Footprint" "" (id 2) (at 236.22 176.53 0)
+      (effects (font (size 1.27 1.27)) hide)
+    )
+    (property "Datasheet" "" (id 3) (at 236.22 176.53 0)
+      (effects (font (size 1.27 1.27)) hide)
+    )
+    (pin "1")
   )
   (symbol (lib_id "Device:R") (at 156.21 125.73 0) (unit 1)
@@
     (pin "2")
   )
-  (symbol (lib_id "74xGxx:74LVC1G17") (at 236.22 172.72 0) (unit 1)
+  (symbol (lib_id "0Local:74LVC1G17QDRY") (at 236.22 172.72 0) (unit 1)
     (in_bom yes) (on_board yes)
     (property "Reference" "U6" (id 0) (at 238.76 166.37 0)
@@
       (effects (font (size 1.27 1.27)) (justify left))
     )
-    (property "Footprint" "Package_TO_SOT_SMD:SOT-886" (id 2) (at 236.22 172.72 0)
-      (effects (font (size 1.27 1.27)) hide)
-    )
-    (property "Datasheet" "http://www.ti.com/lit/sg/scyt129e/scyt129e.pdf" (id 3) (at 236.22 172.72 0)
-      (effects (font (size 1.27 1.27)) hide)
-    )
+    (property "Footprint" "Package_TO_SOT_SMD:SOT-886" (id 2) (at 236.22 181.61 0)
+      (effects (font (size 1.27 1.27)) hide)
+    )
+    (property "Datasheet" "https://www.ti.com/lit/ds/symlink/sn74lvc1g17-q1.pdf" (id 3) (at 236.22 184.15 0)
+      (effects (font (size 1.27 1.27)) hide)
+    )
+    (pin "1")
     (pin "2")
     (pin "3")
     (pin "4")
     (pin "5")
+    (pin "6")
   )
   (symbol (lib_id "Device:R") (at 48.26 54.61 180) (unit 1)
