File: board/1240pi-rompack/cm4_io.kicad_sch (KiCad schematic)
At the start: 4 parts, among them J3 Abracon_ARJM11D7-502-AB-EW2

Commit message: Split connectors out of CM4 footprint.
Parts:
- removed A1: RaspberryPi_CM4, 0Local:RaspberryPi_CM4, symbol 0Local:RaspberryPi_CM4
- added J1: RaspberryPi_CM4_A, 0Local:Hirose_DF40C-100DS-0.4V, symbol 0Local:RaspberryPi_CM4_A
- renumbered J3 to J5
Connections:
- net ETH_LED_G: now also J1.19 (Ethernet_nLED1)
- net ETH_LED_Y: now also J1.17 (Ethernet_nLED2)
- net at J5.1 (TD2+): now also J1.12 (Ethernet_Pair0_P)
- net at J5.10 (TD4-): now also J1.5 (Ethernet_Pair3_N)
- net at J5.2 (TD2-): now also J1.10 (Ethernet_Pair0_N)
- net at J5.3 (TD2+): now also J1.4 (Ethernet_Pair1_P)
- net at J5.4 (TD2-): now also J1.6 (Ethernet_Pair1_N)
- net at J5.7 (TD3+): now also J1.11 (Ethernet_Pair2_P)
- net at J5.8 (TD3-): now also J1.9 (Ethernet_Pair2_N)
- net at J5.9 (TD4+): now also J1.3 (Ethernet_Pair3_P)
Other:
- moved on the sheet: J5, R1, R2
