File: board/1240pi-rompack/host_conp.kicad_sch (KiCad schematic)
At the start: 9 parts, among them P1 CardEdge_ROMPACK, U1 74LVC245A, U2 74LVC245A, U3 74LVC245A, U4 74LVC245A

Commit message: Reroute IO Proc hat again and add buffers on rompack board.
Parts:
- C1, C2, C3, C4: footprint Resistor_SMD:R_0402_1005Metric -> Capacitor_SMD:C_0402_1005Metric
Changed lines of the file:
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@@
     (stroke (width 0) (type default) (color 0 0 0 0))
   )
-  (text "This card-edge connector plugs in to the ROM/RAM Pack socket\nP305 on the Control Processor Board A09. That port was intended\nfor plug-in modules containing ROMs with additional protocol\ndecoding routines or NVRAM for storing configurations. The\nconnector exposes D[0..7] and A[0..15] of the control processor\nbus plus the read and write enables and chip select lines.\n\nThe ROM/RAM Pack as a whole is mapped to 10000h - 1FFFFh\n(64 KB), which is the right size for all 16 of its address lines,\nbut in order to support packs with multiple memory chips the host\nprovides four select lines. To allow for different memory chip sizes,\nthese are decoded from the SEL[0..1] lines, which the pack is\nexpected to connect to the address lines according to its needs.\n\nTo enable packs up to 256 KB, the control processor has an\nalternate addressing mode called PACK EXPAND which decodes\nthe four pack select lines from A[18..19] instead of SEL[0..1].\nIn this mode the selects are mapped as follows:\n\n    ~{CS0}  10000h - 1FFFFh\n    ~{CS1}  50000h - 5FFFFh\n    ~{CS2}  90000h - 9FFFFh\n    ~{CS3}  D0000h - DFFFFh\n\nThis board ties SEL[0..1] low so that ~{CS0} is mapped\nidentically in either addressing mode."
+  (text "This card-edge connector plugs in to the ROM/RAM Pack socket\nP305 on the Control Processor Board A09. That port was intended\nfor plug-in modules containing ROMs with additional protocol\ndecoding routines or NVRAM for storing configurations. The\nconnector exposes D[0..7] and A[0..15] of the control processor\nbus plus the read and write enables and chip select lines.\n\nThe ROM/RAM Pack as a whole is mapped to 10000h - 1FFFFh\n(64 KB), which is the right size for all 16 of its address lines,\nbut in order to support packs with multiple memory chips the host\nprovides four select lines. To allow for different memory chip sizes,\nthese are decoded from the SEL[0..1] lines, which the pack is\nexpected to connect to the address lines according to its needs.\n\nTo enable packs up to 256 KB, the control processor has an\nalternate addressing mode called PACK EXPAND which decodes\nthe four pack select lines from A[18..19] instead of SEL[0..1].\nIn this mode the selects are mapped as follows:\n\n    ~{CS0}  10000h - 1FFFFh\n    ~{CS1}  50000h - 5FFFFh\n    ~{CS2}  90000h - 9FFFFh\n    ~{CS3}  D0000h - DFFFFh\n\nThis board ties SEL[0..1] low so that the address mapping is\nidentical in either addressing mode."
     (at 17.78 198.12 0)
     (effects (font (size 1.27 1.27)) (justify left bottom))
@@
       (effects (font (size 1.27 1.27)) (justify left))
     )
-    (property "Footprint" "Resistor_SMD:R_0402_1005Metric" (id 2) (at 185.42 121.92 0)
+    (property "Footprint" "Capacitor_SMD:C_0402_1005Metric" (id 2) (at 185.42 121.92 0)
       (effects (font (size 1.27 1.27)) hide)
     )
@@
       (effects (font (size 1.27 1.27)) (justify left))
     )
-    (property "Footprint" "Resistor_SMD:R_0402_1005Metric" (id 2) (at 121.92 121.92 0)
+    (property "Footprint" "Capacitor_SMD:C_0402_1005Metric" (id 2) (at 121.92 121.92 0)
       (effects (font (size 1.27 1.27)) hide)
     )
@@
       (effects (font (size 1.27 1.27)) (justify left))
     )
-    (property "Footprint" "Resistor_SMD:R_0402_1005Metric" (id 2) (at 185.42 55.88 0)
+    (property "Footprint" "Capacitor_SMD:C_0402_1005Metric" (id 2) (at 185.42 55.88 0)
       (effects (font (size 1.27 1.27)) hide)
     )
@@
       (effects (font (size 1.27 1.27)) (justify left))
     )
-    (property "Footprint" "Resistor_SMD:R_0402_1005Metric" (id 2) (at 121.92 55.88 0)
-      (effects (font (size 1.27 1.27)) hide)
-    )
+    (property "Footprint" "Capacitor_SMD:C_0402_1005Metric" (id 2) (at 121.92 55.88 0)
+      (effects (font (size 1.27 1.27)) hide)
+    )
