File: board/1240pi-rompack/host_iop.kicad_sch (KiCad schematic)
At the start: 9 parts, among them J6 62684-50210, U5 74LVC245A, U6 74LVC245A, U7 74LVC245A, U8 74LVC245A

Commit message: Add description to IO proc interface.
Parts:
- added R? (x2): 10k, symbol Device:R
Connections:
- net +3V3: now also R?.1, R?.1
- net ~{BUSACK}: now also U5.1 (A->B), U6.1 (A->B)
- net ~{IORQ}: now also R?.2
- net ~{IDOUT}: now reaches U7.1 (A->B)
- net ~{IDOUT}: now also R?.2
Other:
- note added: "The flat flex cable connects to the IO Processor Mod board, which taps all 40 pins of the Z80 on the IO Processor board. The interface has two modes, observing and controlling. In observing mode the digital lines are all high-impedance inputs and the FPGA monitors the activity on the bus. In controlling mode we put the Z80 in DMA mode, which is not used by the host machine, and the FPGA takes con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"
- note added: "~{HALT}, ~{M1}, ~{RFSH}, and ~{BUSACK} are outputs of the Z80 which are not released in DMA mode. We have no reason to drive them. ~{IORQ} is a Z80 output which is released in DMA mode but is not used on the host board so we have no reason to drive it. We pull it high to avoid a floating input on our buffer when the Z80 is in DMA mode. ~{CLK} is a Z80 input which is always driven by the host boar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"
Changed lines of the file:
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@@
+    (stroke (width 0) (type default) (color 0 0 0 0))
+  )
+  (wire (pts (xy 76.2 114.3) (xy 83.82 114.3))
     (stroke (width 0) (type default) (color 0 0 0 0))
   )
@@
     (stroke (width 0) (type default) (color 0 0 0 0))
   )
+  (wire (pts (xy 147.32 50.8) (xy 139.7 50.8))
+    (stroke (width 0) (type default) (color 0 0 0 0))
+  )
   (wire (pts (xy 172.72 93.98) (xy 182.88 93.98))
     (stroke (width 0) (type default) (color 0 0 0 0))
@@
     (stroke (width 0) (type default) (color 0 0 0 0))
   )
+  (wire (pts (xy 208.28 149.86) (xy 220.98 149.86))
+    (stroke (width 0) (type default) (color 0 0 0 0))
+  )
   (wire (pts (xy 180.34 33.02) (xy 172.72 33.02))
     (stroke (width 0) (type default) (color 0 0 0 0))
@@
     (stroke (width 0) (type default) (color 0 0 0 0))
   )
+  (wire (pts (xy 190.5 147.32) (xy 190.5 149.86))
+    (stroke (width 0) (type default) (color 0 0 0 0))
+  )
   (wire (pts (xy 48.26 121.92) (xy 58.42 121.92))
     (stroke (width 0) (type default) (color 0 0 0 0))
@@
     (stroke (width 0) (type default) (color 0 0 0 0))
   )
+  (wire (pts (xy 83.82 50.8) (xy 76.2 50.8))
+    (stroke (width 0) (type default) (color 0 0 0 0))
+  )
   (wire (pts (xy 160.02 127) (xy 160.02 129.54))
     (stroke (width 0) (type default) (color 0 0 0 0))
   )
+  (wire (pts (xy 190.5 149.86) (xy 203.2 149.86))
+    (stroke (width 0) (type default) (color 0 0 0 0))
+  )
   (wire (pts (xy 48.26 68.58) (xy 58.42 68.58))
     (stroke (width 0) (type default) (color 0 0 0 0))
@@
     (stroke (width 0) (type default) (color 0 0 0 0))
   )
+  (wire (pts (xy 208.28 147.32) (xy 208.28 149.86))
+    (stroke (width 0) (type default) (color 0 0 0 0))
+  )
   (wire (pts (xy 172.72 96.52) (xy 182.88 96.52))
     (stroke (width 0) (type default) (color 0 0 0 0))
   )
+  (text "The flat flex cable connects to the IO Processor Mod board,\nwhich taps all 40 pins of the Z80 on the IO Processor board.\n\nThe interface has two modes, observing and controlling.\nIn observing mode the digital lines are all high-impedance\ninputs and the FPGA monitors the activity on the bus.\nIn controlling mode we put the Z80 in DMA mode, which is not\nused by the host machine, and the FPGA takes control of the bus.\n\nTo enter controlling mode we assert the ~{BUSREQ} signal. At the\nend of its current machine cycle the Z80 will enter DMA mode and\nrelease the bus for external use by setting all of its bus IOs\n(A[0..15], D[0..7], ~{RD}, ~{WR}, ~{MREQ}, and ~{IORQ}) to high impedance.\nWhen the Z80 has released the bus it will assert ~{BUSACK}.\n\nThe buffers for A[0..15], ~{RD}, ~{WR}, and ~{MREQ} switch direction on\n~{BUSACK} because in controlling mode we always drive those signals.\nThe FPGA controls the direction of the D[0..7] buffer because it\ndepends on both the interface mode and the read/write mode."
+    (at 25.4 190.5 0)
+    (effects (font (size 1.27 1.27)) (justify left bottom))
+  )
+  (text "~{HALT}, ~{M1}, ~{RFSH}, and ~{BUSACK} are outputs of the Z80 which are not\nreleased in DMA mode. We have no reason to drive them.\n\n~{IORQ} is a Z80 output which is released in DMA mode but is not used\non the host board so we have no reason to drive it. We pull it high\nto avoid a floating input on our buffer when the Z80 is in DMA mode.\n\n~{CLK} is a Z80 input which is always driven by the host board.\n\n~{RESET}, ~{INT}, and ~{WAIT} are wired-OR Z80 inputs which are generated\nby the host board. We may also want to drive them low sometimes.\n\n~{BUSREQ} and ~{NMI} are Z80 inputs which are not used by the host board.\nWe drive them but have no reason to monitor them."
+    (at 101.6 190.5 0)
+    (effects (font (size 1.27 1.27)) (justify left bottom))
+  )
   (label "ID7" (at 116.84 109.22 180)
     (effects (font (size 1.27 1.27)) (justify right bottom))
@@
     (effects (font (size 1.27 1.27)) (justify right bottom))
   )
+  (label "~{IDOUT}" (at 203.2 149.86 180)
+    (effects (font (size 1.27 1.27)) (justify right bottom))
+  )
   (label "A9" (at 139.7 30.48 0)
     (effects (font (size 1.27 1.27)) (justify left bottom))
@@
     (effects (font (size 1.27 1.27)) (justify right bottom))
   )
+  (label "~{BUSACK}" (at 76.2 50.8 0)
+    (effects (font (size 1.27 1.27)) (justify left bottom))
+  )
   (label "IA14" (at 180.34 43.18 180)
     (effects (font (size 1.27 1.27)) (justify right bottom))
@@
     (effects (font (size 1.27 1.27)) (justify right bottom))
   )
+  (label "~{IORQ}" (at 220.98 149.86 180)
+    (effects (font (size 1.27 1.27)) (justify right bottom))
+  )
   (label "A7" (at 76.2 27.94 0)
     (effects (font (size 1.27 1.27)) (justify left bottom))
@@
     (effects (font (size 1.27 1.27)) (justify right bottom))
   )
+  (label "~{IDOUT}" (at 76.2 114.3 0)
+    (effects (font (size 1.27 1.27)) (justify left bottom))
+  )
   (label "~{IRFSH}" (at 182.88 99.06 180)
     (effects (font (size 1.27 1.27)) (justify right bottom))
@@
   (label "D7" (at 58.42 93.98 180)
     (effects (font (size 1.27 1.27)) (justify right bottom))
+  )
+  (label "~{BUSACK}" (at 139.7 50.8 0)
+    (effects (font (size 1.27 1.27)) (justify left bottom))
   )
   (label "A15" (at 139.7 45.72 0)
@@
     )
     (pin "1")
+  )
+  (symbol (lib_id "Device:R") (at 190.5 143.51 0) (unit 1)
+    (in_bom yes) (on_board yes)
+    (property "Reference" "R?" (id 0) (at 192.532 143.51 90))
+    (property "Value" "10k" (id 1) (at 190.5 143.51 90))
+    (property "Footprint" "" (id 2) (at 188.722 143.51 90)
+      (effects (font (size 1.27 1.27)) hide)
+    )
+    (property "Datasheet" "~" (id 3) (at 190.5 143.51 0)
+      (effects (font (size 1.27 1.27)) hide)
+    )
+    (pin "1")
+    (pin "2")
   )
   (symbol (lib_id "74xx:74LS245") (at 96.52 104.14 0) (unit 1)
@@
     (pin "1")
   )
+  (symbol (lib_id "Device:R") (at 208.28 143.51 0) (unit 1)
+    (in_bom yes) (on_board yes)
+    (property "Reference" "R?" (id 0) (at 210.312 143.51 90))
+    (property "Value" "10k" (id 1) (at 208.28 143.51 90))
+    (property "Footprint" "" (id 2) (at 206.502 143.51 90)
+      (effects (font (size 1.27 1.27)) hide)
+    )
+    (property "Datasheet" "~" (id 3) (at 208.28 143.51 0)
+      (effects (font (size 1.27 1.27)) hide)
+    )
+    (pin "1")
+    (pin "2")
+  )
   (symbol (lib_id "power:GND") (at 96.52 129.54 0) (unit 1)
     (in_bom yes) (on_board yes) (fields_autoplaced)
@@
     (pin "1")
   )
+  (symbol (lib_id "power:+3V3") (at 208.28 139.7 0) (unit 1)
+    (in_bom yes) (on_board yes)
+    (property "Reference" "#PWR?" (id 0) (at 208.28 143.51 0)
+      (effects (font (size 1.27 1.27)) hide)
+    )
+    (property "Value" "+3V3" (id 1) (at 208.28 136.144 0))
+    (property "Footprint" "" (id 2) (at 208.28 139.7 0)
+      (effects (font (size 1.27 1.27)) hide)
+    )
+    (property "Datasheet" "" (id 3) (at 208.28 139.7 0)
+      (effects (font (size 1.27 1.27)) hide)
+    )
+    (pin "1")
+  )
   (symbol (lib_id "power:GND") (at 172.72 121.92 0) (unit 1)
     (in_bom yes) (on_board yes) (fields_autoplaced)
@@
       (effects (font (size 1.27 1.27)) hide)
     )
+    (pin "1")
+  )
+  (symbol (lib_id "power:+3V3") (at 190.5 139.7 0) (unit 1)
+    (in_bom yes) (on_board yes)
+    (property "Reference" "#PWR?" (id 0) (at 190.5 143.51 0)
+      (effects (font (size 1.27 1.27)) hide)
+    )
+    (property "Value" "+3V3" (id 1) (at 190.5 136.144 0))
+    (property "Footprint" "" (id 2) (at 190.5 139.7 0)
+      (effects (font (size 1.27 1.27)) hide)
+    )
+    (property "Datasheet" "" (id 3) (at 190.5 139.7 0)
+      (effects (font (size 1.27 1.27)) hide)
+    )

Commit message: Reroute IO Proc hat again and add buffers on rompack board.
Parts:
- removed R?: 10k, symbol Device:R
- added C12: 100n, Capacitor_SMD:C_0402_1005Metric, symbol Device:C_Small
- added U10: 74LS126, symbol 74xx:74LS126
- added U9: 74LVC245A, 0Local:Nexperia_SOT764-1, symbol 74xx:74LS245
- C5, C6, C7, C8: footprint Resistor_SMD:R_0402_1005Metric -> Capacitor_SMD:C_0402_1005Metric
- R3: renamed from R?; footprint (none) -> Resistor_SMD:R_0402_1005Metric
Connections:
- net +3V3: now also C12.1, U9.20 (VCC)
- net GND: now also C12.2, U9.10 (GND), U9.19 (CE), U9.2 (A0), U9.3 (A1), U9.7 (A5), U9.9 (A7)
- net ~{BUSACK}: now also U9.1 (A->B)
- net ~{IIORQ}: now also U9.12 (B6); no longer U8.17 (B1)
- net ~{IORQ}: now also J6.31 (~{IORQ}), U9.8 (A6); no longer J6.39 (~{IORQ}), U8.3 (A1)
- net ~{MREQ}: now also U9.5 (A3)
- net ~{RD}: now also U9.6 (A4)
- net ~{RESET}: now also J6.39 (~{RESET}), U8.3 (A1); no longer J6.31 (~{RESET})
- net ~{WR}: now also U9.4 (A2)
- new net ~{IMREQ}: U9.15 (B3)
- new net ~{IRD}: U9.14 (B4)
- new net ~{IRESET}: U8.17 (B1)
- new net ~{IWR}: U9.16 (B2)
- no-connect marks 1 -> 5
Other:
- note added: "42 pins to FPGA"
- note added: "Drive ~{RESET}, ~{INT}, ~{WAIT}, ~{BUSREQ}, ~{NMI}"
- note added: "~{HALT}, ~{M1}, ~{RFSH}, and ~{BUSACK} are outputs of the Z80 which are not released in DMA mode. We have no reason to drive them. ~{CLK} is a Z80 input which is always driven by the host board. ~{RESET}, ~{INT}, and ~{WAIT} are wired-OR Z80 inputs which are generated by the host board. We may also want to drive them low sometimes. ~{BUSREQ} and ~{NMI} are Z80 inputs which are not used by the hos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"
- note removed: "~{HALT}, ~{M1}, ~{RFSH}, and ~{BUSACK} are outputs of the Z80 which are not released in DMA mode. We have no reason to drive them. ~{IORQ} is a Z80 output which is released in DMA mode but is not used on the host board so we have no reason to drive it. We pull it high to avoid a floating input on our buffer when the Z80 is in DMA mode. ~{CLK} is a Z80 input which is always driven by the host boar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"
- moved on the sheet: C6, C8, R3, U6, U8
