File: board/1240pi-io-proc-hat/1240pi-io-proc-hat.kicad_sch (KiCad schematic)
At the start: 6 parts, among them J1 62684-50210, J2 SFV10R-1ST, P445 Header, U445 Z80

Commit message: Reroute IO Proc hat again and add buffers on rompack board.
Connections:
- net ~{IORQ}: now also J1.20 (Pin_20); no longer J1.12 (Pin_12)
- net ~{RESET}: now also J1.12 (Pin_12); no longer J1.20 (Pin_20)
Changed lines of the file:
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@@
     (effects (font (size 1.27 1.27)) (justify left bottom))
   )
-  (label "~{IORQ}" (at 203.2 104.14 0)
+  (label "~{IORQ}" (at 203.2 124.46 0)
     (effects (font (size 1.27 1.27)) (justify left bottom))
   )
@@
     (effects (font (size 1.27 1.27)) (justify left bottom))
   )
-  (label "~{RESET}" (at 203.2 124.46 0)
+  (label "~{RESET}" (at 203.2 104.14 0)
     (effects (font (size 1.27 1.27)) (justify left bottom))
   )
